File: Electronics/Fire-Sensor.brd (EAGLE design)
At the start: 160 x 100 mm, 8 parts, among them IC1 REG1117

Commit message: Regular Commit - New examples
Parts:
- removed THERMOMETER: LM35CZ, lm35:TO92
Connections:
- removed net N$6: ARDUINO.A5, THERMOMETER.2
- net +5V: no longer THERMOMETER.1
- net GND: no longer THERMOMETER.3
Routing:
- net N$6: track 13.3 -> 0.00 mm
- net +5V: track 51.4 -> 42.5 mm
- net GND: track 163.1 -> 160.6 mm
Changed lines of the file:
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@@
 </element>
 <element name="LDR" library="photo-elements" package="T0-46-A10XX" value="A1050_09" x="34.29" y="31.75"/>
-<element name="THERMOMETER" library="lm35" package="TO92" value="LM35CZ" x="34.29" y="50.8" rot="R180"/>
 <element name="DHT11" library="con-molex" package="KK-156-3" value="" x="34.29" y="64.77">
 <attribute name="OC_NEWARK" value="unknown" x="53.34" y="15.24" size="1.778" layer="27" display="off"/>
@@
 <contactref element="ARDUINO" pad="GND_USB"/>
 <contactref element="IC1" pad="1"/>
-<contactref element="THERMOMETER" pad="3"/>
 <contactref element="DHT11" pad="3"/>
 <contactref element="ESP8266" pad="7"/>
@@
 <wire x1="67.41" y1="61.38" x2="67.41" y2="62.23" width="1.27" layer="16"/>
 <wire x1="67.41" y1="62.23" x2="58.42" y2="62.23" width="1.27" layer="16"/>
-<wire x1="33.02" y1="50.8" x2="30.48" y2="50.8" width="1.27" layer="16"/>
 <wire x1="30.48" y1="50.8" x2="30.48" y2="45.72" width="1.27" layer="16"/>
 <wire x1="38.25" y1="64.77" x2="38.25" y2="71.12" width="1.27" layer="16"/>
@@
 <signal name="+5V">
 <contactref element="LDR" pad="2"/>
-<contactref element="THERMOMETER" pad="1"/>
 <contactref element="DHT11" pad="1"/>
 <contactref element="ARDUINO" pad="5V"/>
@@
 <wire x1="39.37" y1="33.02" x2="39.37" y2="36.83" width="1.27" layer="16"/>
 <wire x1="30.48" y1="64.77" x2="30.33" y2="64.77" width="1.27" layer="16"/>
-<wire x1="35.56" y1="50.8" x2="40.64" y2="50.8" width="1.27" layer="16"/>
 <via x="40.64" y="50.8" extent="1-16" drill="0.6" shape="square"/>
 <wire x1="40.64" y1="50.8" x2="40.64" y2="36.83" width="1.27" layer="1"/>
 <wire x1="30.48" y1="64.77" x2="30.48" y2="54.61" width="1.27" layer="16"/>
 <wire x1="30.48" y1="54.61" x2="35.56" y2="54.61" width="1.27" layer="16"/>
-<wire x1="35.56" y1="54.61" x2="35.56" y2="50.8" width="1.27" layer="16"/>
 <via x="40.64" y="36.83" extent="1-16" drill="0.6" shape="square"/>
+<wire x1="40.64" y1="50.8" x2="35.56" y2="54.61" width="0" layer="19" extent="16-16"/>
 </signal>
 <signal name="H/T">
@@
 <wire x1="60.96" y1="41.91" x2="55.88" y2="41.91" width="1.27" layer="16"/>
 </signal>
-<signal name="N$6">
-<contactref element="THERMOMETER" pad="2"/>
-<contactref element="ARDUINO" pad="A5"/>
-<wire x1="39.37" y1="48.895" x2="39.37" y2="44.45" width="1.27" layer="16"/>
-<wire x1="39.37" y1="44.45" x2="43.18" y2="44.45" width="1.27" layer="16"/>
-<wire x1="39.37" y1="48.895" x2="34.29" y2="48.895" width="1.27" layer="16"/>
-</signal>
 <signal name="VCC">
