File: Electronics/Fire-Sensor.sch (EAGLE design)
At the start: 8 parts, among them IC1 REG1117

Commit message: Regular Commit - New examples
Parts:
- removed THERMOMETER: LM35CZ, lm35:LM35CZ
Connections:
- removed net N$6: ARDUINO.A5, THERMOMETER.VO
- net +5V: no longer THERMOMETER.+VS
- net GND: no longer THERMOMETER.GND
Changed lines of the file:
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@@
 <part name="IC1" library="burr-brown" deviceset="REG1117" device=""/>
 <part name="LDR" library="photo-elements" deviceset="A10" device="" technology="50_09"/>
-<part name="THERMOMETER" library="lm35" deviceset="LM35" device="CZ"/>
 <part name="DHT11" library="con-molex" deviceset="KK-156-3" device=""/>
 <part name="GND1" library="supply1" deviceset="GND" device=""/>
 <part name="GND2" library="supply1" deviceset="GND" device=""/>
-<part name="GND3" library="supply1" deviceset="GND" device=""/>
 <part name="GND4" library="supply1" deviceset="GND" device=""/>
 <part name="GND5" library="supply1" deviceset="GND" device=""/>
@@
 <part name="P+6" library="supply1" deviceset="+5V" device=""/>
 <part name="P+7" library="supply1" deviceset="+5V" device=""/>
-<part name="P+8" library="supply1" deviceset="+5V" device=""/>
 <part name="P+9" library="supply1" deviceset="+5V" device=""/>
 <part name="+3V2" library="supply1" deviceset="+3V3" device=""/>
@@
 <instance part="IC1" gate="G$1" x="160.02" y="86.36"/>
 <instance part="LDR" gate="G$1" x="7.62" y="81.28" rot="R180"/>
-<instance part="THERMOMETER" gate="G$1" x="58.42" y="66.04"/>
 <instance part="DHT11" gate="-1" x="27.94" y="68.58"/>
 <instance part="DHT11" gate="-2" x="27.94" y="66.04"/>
@@
 <instance part="GND1" gate="1" x="160.02" y="66.04"/>
 <instance part="GND2" gate="1" x="96.52" y="5.08"/>
-<instance part="GND3" gate="1" x="58.42" y="53.34"/>
 <instance part="GND4" gate="1" x="22.86" y="53.34"/>
 <instance part="GND5" gate="1" x="7.62" y="53.34"/>
@@
 <instance part="P+6" gate="1" x="99.06" y="81.28"/>
 <instance part="P+7" gate="1" x="7.62" y="91.44"/>
-<instance part="P+8" gate="1" x="43.18" y="91.44"/>
 <instance part="P+9" gate="1" x="22.86" y="91.44"/>
 <instance part="+3V2" gate="G$1" x="177.8" y="40.64"/>
@@
 <pinref part="IC1" gate="G$1" pin="GND"/>
 <wire x1="160.02" y1="68.58" x2="160.02" y2="73.66" width="0.1524" layer="91"/>
-</segment>
-<segment>
-<pinref part="THERMOMETER" gate="G$1" pin="GND"/>
-<pinref part="GND3" gate="1" pin="GND"/>
-<wire x1="58.42" y1="55.88" x2="58.42" y2="58.42" width="0.1524" layer="91"/>
 </segment>
 <segment>
@@
 </segment>
 <segment>
-<pinref part="P+8" gate="1" pin="+5V"/>
-<pinref part="THERMOMETER" gate="G$1" pin="+VS"/>
-<wire x1="43.18" y1="88.9" x2="43.18" y2="66.04" width="0.1524" layer="91"/>
-<wire x1="43.18" y1="66.04" x2="48.26" y2="66.04" width="0.1524" layer="91"/>
-</segment>
-<segment>
 <pinref part="DHT11" gate="-1" pin="S"/>
 <pinref part="P+9" gate="1" pin="+5V"/>
@@
 </segment>
 </net>
-<net name="N$6" class="0">
-<segment>
-<pinref part="THERMOMETER" gate="G$1" pin="VO"/>
-<wire x1="68.58" y1="66.04" x2="71.12" y2="66.04" width="0.1524" layer="91"/>
-<pinref part="ARDUINO" gate="G$1" pin="A5"/>
-<wire x1="78.74" y1="43.18" x2="71.12" y2="43.18" width="0.1524" layer="91"/>
-<wire x1="71.12" y1="43.18" x2="71.12" y2="66.04" width="0.1524" layer="91"/>
-</segment>
-</net>
